Commit message: feat: consolidate closed-loop navigation stack

File: modubot_ws/src/modubot_model_description/urdf/modubot_model.xacro (robot description, xacro)
@@ -11,5 +11,5 @@
     <origin xyz="0 0 0" rpy="0 0 0"/>
     <geometry>
-      <mesh filename="file://$(find modubot_model_description)/meshes/base_link.stl" scale="0.001 0.001 0.001"/>
+      <mesh filename="package://modubot_model_description/meshes/base_link.stl" scale="0.001 0.001 0.001"/>
     </geometry>
     <material name="silver"/>
@@ -18,5 +18,5 @@
     <origin xyz="0 0 0" rpy="0 0 0"/>
     <geometry>
-      <mesh filename="file://$(find modubot_model_description)/meshes/base_link.stl" scale="0.001 0.001 0.001"/>
+      <mesh filename="package://modubot_model_description/meshes/base_link.stl" scale="0.001 0.001 0.001"/>
     </geometry>
   </collision>
@@ -31,5 +31,5 @@
     <origin xyz="-0.002507 -0.004307 -0.219668" rpy="0 0 0"/>
     <geometry>
-      <mesh filename="file://$(find modubot_model_description)/meshes/lidar_1.stl" scale="0.001 0.001 0.001"/>
+      <mesh filename="package://modubot_model_description/meshes/lidar_1.stl" scale="0.001 0.001 0.001"/>
     </geometry>
     <material name="silver"/>
@@ -38,5 +38,5 @@
     <origin xyz="-0.002507 -0.004307 -0.219668" rpy="0 0 0"/>
     <geometry>
-      <mesh filename="file://$(find modubot_model_description)/meshes/lidar_1.stl" scale="0.001 0.001 0.001"/>
+      <mesh filename="package://modubot_model_description/meshes/lidar_1.stl" scale="0.001 0.001 0.001"/>
     </geometry>
   </collision>
@@ -51,5 +51,5 @@
     <origin xyz="0.375122 0.16578 -0.047978" rpy="0 0 0"/>
     <geometry>
-      <mesh filename="file://$(find modubot_model_description)/meshes/right_caster_1.stl" scale="0.001 0.001 0.001"/>
+      <mesh filename="package://modubot_model_description/meshes/right_caster_1.stl" scale="0.001 0.001 0.001"/>
     </geometry>
     <material name="silver"/>
@@ -58,5 +58,5 @@
     <origin xyz="0.375122 0.16578 -0.047978" rpy="0 0 0"/>
     <geometry>
-      <mesh filename="file://$(find modubot_model_description)/meshes/right_caster_1.stl" scale="0.001 0.001 0.001"/>
+      <mesh filename="package://modubot_model_description/meshes/right_caster_1.stl" scale="0.001 0.001 0.001"/>
     </geometry>
   </collision>
@@ -71,5 +71,5 @@
     <origin xyz="0.375122 -0.16422 -0.047978" rpy="0 0 0"/>
     <geometry>
-      <mesh filename="file://$(find modubot_model_description)/meshes/left_caster_1.stl" scale="0.001 0.001 0.001"/>
+      <mesh filename="package://modubot_model_description/meshes/left_caster_1.stl" scale="0.001 0.001 0.001"/>
     </geometry>
     <material name="silver"/>
@@ -78,5 +78,5 @@
     <origin xyz="0.375122 -0.16422 -0.047978" rpy="0 0 0"/>
     <geometry>
-      <mesh filename="file://$(find modubot_model_description)/meshes/left_caster_1.stl" scale="0.001 0.001 0.001"/>
+      <mesh filename="package://modubot_model_description/meshes/left_caster_1.stl" scale="0.001 0.001 0.001"/>
     </geometry>
   </collision>
@@ -91,5 +91,5 @@
     <origin xyz="0.001398 0.100604 -0.060978" rpy="0 0 0"/>
     <geometry>
-      <mesh filename="file://$(find modubot_model_description)/meshes/right_wheel_1.stl" scale="0.001 0.001 0.001"/>
+      <mesh filename="package://modubot_model_description/meshes/right_wheel_1.stl" scale="0.001 0.001 0.001"/>
     </geometry>
     <material name="silver"/>
@@ -98,5 +98,5 @@
     <origin xyz="0.001398 0.100604 -0.060978" rpy="0 0 0"/>
     <geometry>
-      <mesh filename="file://$(find modubot_model_description)/meshes/right_wheel_1.stl" scale="0.001 0.001 0.001"/>
+      <mesh filename="package://modubot_model_description/meshes/right_wheel_1.stl" scale="0.001 0.001 0.001"/>
     </geometry>
   </collision>
@@ -111,5 +111,5 @@
     <origin xyz="0.001398 -0.106396 -0.060978" rpy="0 0 0"/>
     <geometry>
-      <mesh filename="file://$(find modubot_model_description)/meshes/left_wheel_1.stl" scale="0.001 0.001 0.001"/>
+      <mesh filename="package://modubot_model_description/meshes/left_wheel_1.stl" scale="0.001 0.001 0.001"/>
     </geometry>
     <material name="silver"/>
@@ -118,5 +118,5 @@
     <origin xyz="0.001398 -0.106396 -0.060978" rpy="0 0 0"/>
     <geometry>
-      <mesh filename="file://$(find modubot_model_description)/meshes/left_wheel_1.stl" scale="0.001 0.001 0.001"/>
+      <mesh filename="package://modubot_model_description/meshes/left_wheel_1.stl" scale="0.001 0.001 0.001"/>
     </geometry>
   </collision>
@@ -131,5 +131,5 @@
     <origin xyz="0.101 -0.002 -1.486512" rpy="0 0 0"/>
     <geometry>
-      <mesh filename="file://$(find modubot_model_description)/meshes/camera_1.stl" scale="0.001 0.001 0.001"/>
+      <mesh filename="package://modubot_model_description/meshes/camera_1.stl" scale="0.001 0.001 0.001"/>
     </geometry>
     <material name="silver"/>
@@ -138,5 +138,5 @@
     <origin xyz="0.101 -0.002 -1.486512" rpy="0 0 0"/>
     <geometry>
-      <mesh filename="file://$(find modubot_model_description)/meshes/camera_1.stl" scale="0.001 0.001 0.001"/>
+      <mesh filename="package://modubot_model_description/meshes/camera_1.stl" scale="0.001 0.001 0.001"/>
     </geometry>
   </collision>

Commit message: feat: add DC first-floor Nav2 simulation

File: modubot_ws/src/modubot_model_description/urdf/modubot_model.xacro (robot description, xacro)
@@ -2,4 +2,5 @@
 <robot name="modubot_model" xmlns:xacro="http://www.ros.org/wiki/xacro">
 <xacro:include filename="$(find modubot_model_description)/urdf/materials.xacro" />
+<xacro:arg name="mesh_prefix" default="package://modubot_model_description/meshes" />
 <link name="base_link">
   <inertial>
@@ -11,5 +12,5 @@
     <origin xyz="0 0 0" rpy="0 0 0"/>
     <geometry>
-      <mesh filename="package://modubot_model_description/meshes/base_link.stl" scale="0.001 0.001 0.001"/>
+      <mesh filename="$(arg mesh_prefix)/base_link.stl" scale="0.001 0.001 0.001"/>
     </geometry>
     <material name="silver"/>
@@ -18,5 +19,5 @@
     <origin xyz="0 0 0" rpy="0 0 0"/>
     <geometry>
-      <mesh filename="package://modubot_model_description/meshes/base_link.stl" scale="0.001 0.001 0.001"/>
+      <mesh filename="$(arg mesh_prefix)/base_link.stl" scale="0.001 0.001 0.001"/>
     </geometry>
   </collision>
@@ -31,5 +32,5 @@
     <origin xyz="-0.002507 -0.004307 -0.219668" rpy="0 0 0"/>
     <geometry>
-      <mesh filename="package://modubot_model_description/meshes/lidar_1.stl" scale="0.001 0.001 0.001"/>
+      <mesh filename="$(arg mesh_prefix)/lidar_1.stl" scale="0.001 0.001 0.001"/>
     </geometry>
     <material name="silver"/>
@@ -38,5 +39,5 @@
     <origin xyz="-0.002507 -0.004307 -0.219668" rpy="0 0 0"/>
     <geometry>
-      <mesh filename="package://modubot_model_description/meshes/lidar_1.stl" scale="0.001 0.001 0.001"/>
+      <mesh filename="$(arg mesh_prefix)/lidar_1.stl" scale="0.001 0.001 0.001"/>
     </geometry>
   </collision>
@@ -51,5 +52,5 @@
     <origin xyz="0.375122 0.16578 -0.047978" rpy="0 0 0"/>
     <geometry>
-      <mesh filename="package://modubot_model_description/meshes/right_caster_1.stl" scale="0.001 0.001 0.001"/>
+      <mesh filename="$(arg mesh_prefix)/right_caster_1.stl" scale="0.001 0.001 0.001"/>
     </geometry>
     <material name="silver"/>
@@ -58,5 +59,5 @@
     <origin xyz="0.375122 0.16578 -0.047978" rpy="0 0 0"/>
     <geometry>
-      <mesh filename="package://modubot_model_description/meshes/right_caster_1.stl" scale="0.001 0.001 0.001"/>
+      <mesh filename="$(arg mesh_prefix)/right_caster_1.stl" scale="0.001 0.001 0.001"/>
     </geometry>
   </collision>
@@ -71,5 +72,5 @@
     <origin xyz="0.375122 -0.16422 -0.047978" rpy="0 0 0"/>
     <geometry>
-      <mesh filename="package://modubot_model_description/meshes/left_caster_1.stl" scale="0.001 0.001 0.001"/>
+      <mesh filename="$(arg mesh_prefix)/left_caster_1.stl" scale="0.001 0.001 0.001"/>
     </geometry>
     <material name="silver"/>
@@ -78,5 +79,5 @@
     <origin xyz="0.375122 -0.16422 -0.047978" rpy="0 0 0"/>
     <geometry>
-      <mesh filename="package://modubot_model_description/meshes/left_caster_1.stl" scale="0.001 0.001 0.001"/>
+      <mesh filename="$(arg mesh_prefix)/left_caster_1.stl" scale="0.001 0.001 0.001"/>
     </geometry>
   </collision>
@@ -91,5 +92,5 @@
     <origin xyz="0.001398 0.100604 -0.060978" rpy="0 0 0"/>
     <geometry>
-      <mesh filename="package://modubot_model_description/meshes/right_wheel_1.stl" scale="0.001 0.001 0.001"/>
+      <mesh filename="$(arg mesh_prefix)/right_wheel_1.stl" scale="0.001 0.001 0.001"/>
     </geometry>
     <material name="silver"/>
@@ -98,5 +99,5 @@
     <origin xyz="0.001398 0.100604 -0.060978" rpy="0 0 0"/>
     <geometry>
-      <mesh filename="package://modubot_model_description/meshes/right_wheel_1.stl" scale="0.001 0.001 0.001"/>
+      <mesh filename="$(arg mesh_prefix)/right_wheel_1.stl" scale="0.001 0.001 0.001"/>
     </geometry>
   </collision>
@@ -111,5 +112,5 @@
     <origin xyz="0.001398 -0.106396 -0.060978" rpy="0 0 0"/>
     <geometry>
-      <mesh filename="package://modubot_model_description/meshes/left_wheel_1.stl" scale="0.001 0.001 0.001"/>
+      <mesh filename="$(arg mesh_prefix)/left_wheel_1.stl" scale="0.001 0.001 0.001"/>
     </geometry>
     <material name="silver"/>
@@ -118,5 +119,5 @@
     <origin xyz="0.001398 -0.106396 -0.060978" rpy="0 0 0"/>
     <geometry>
-      <mesh filename="package://modubot_model_description/meshes/left_wheel_1.stl" scale="0.001 0.001 0.001"/>
+      <mesh filename="$(arg mesh_prefix)/left_wheel_1.stl" scale="0.001 0.001 0.001"/>
     </geometry>
   </collision>
@@ -131,5 +132,5 @@
     <origin xyz="0.101 -0.002 -1.486512" rpy="0 0 0"/>
     <geometry>
-      <mesh filename="package://modubot_model_description/meshes/camera_1.stl" scale="0.001 0.001 0.001"/>
+      <mesh filename="$(arg mesh_prefix)/camera_1.stl" scale="0.001 0.001 0.001"/>
     </geometry>
     <material name="silver"/>
@@ -138,5 +139,5 @@
     <origin xyz="0.101 -0.002 -1.486512" rpy="0 0 0"/>
     <geometry>
-      <mesh filename="package://modubot_model_description/meshes/camera_1.stl" scale="0.001 0.001 0.001"/>
+      <mesh filename="$(arg mesh_prefix)/camera_1.stl" scale="0.001 0.001 0.001"/>
     </geometry>
   </collision>
